File: DAC.sch (EAGLE design)
At the start: 89 parts, among them IC1 LM2662, IC2 PCM1793, IC3 OPA2134PA, IC4 LMH6643, J1 USBSMD, J2 RCJ-21XXMILL, U1 LDO-TPS78233, U2 PCM2707, Y1 12MHz/20pF

Commit message: 2.5mm jack was placed by mistake
Parts:
- J3: device SparkFun-Connectors:AUDIO-JACK2.5MM -> SparkFun-Connectors:AUDIO-JACKPTH
Changed lines of the file:
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@@
 <part name="R24" library="SparkFun-Resistors" deviceset="RESISTOR" device="PTH-1/4W" value="1.8k"/>
 <part name="C43" library="SparkFun-Capacitors" deviceset="CAP" device="PTH" value="100pF"/>
-<part name="J3" library="SparkFun-Connectors" deviceset="AUDIO-JACK" device="2.5MM"/>
+<part name="J3" library="SparkFun-Connectors" deviceset="AUDIO-JACK" device="PTH"/>
 <part name="R28" library="SparkFun-Resistors" deviceset="RESISTOR" device="PTH-1/4W" value="3.3k"/>
 <part name="R27" library="SparkFun-Resistors" deviceset="RESISTOR" device="PTH-1/4W" value="1.8k"/>
